File: Hardware/SparkFun_CAN-Bus_Shield.brd (EAGLE design)
At the start: 53.3 x 59.7 mm, 48 parts, among them Q1 16MHz, U1 USD-SOCKETNEW, U2 ARDUINO_R3_SHIELD, U3 JST_VERTICAL, U4 MCP2515, U5 MCP2551, U6 HEX_CONVERTER, X1 DB9 Plug

Commit message: Updating to new uSD footprint, minor QC cleanup on schematic
Parts:
- FRAME1: value (none) -> FRAME-LETTER
- FRAME2: value (none) -> FRAME-LETTERNO_PACKAGE
- U1: value USD-SOCKETNEW -> USD-SOCKET; device SparkFun-Connectors:MICRO-SD-SOCKET-PP -> SparkFun-Connectors:MICROSD_1:1
- moved U1 14.0 mm to (30.5, 16.5)
Other:
- board text added: "Sukkin Pang"
