File: Hardware/SparkFun_CAN-Bus_Shield.brd (EAGLE design)
At the start: 53.3 x 59.7 mm, 48 parts, among them Q1 16MHz, U1 USD-SOCKET, U2 ARDUINO_R3_SHIELD, U3 JST_VERTICAL, U4 MCP2515, U5 MCP2551, U6 HEX_CONVERTER, X1 DB9 Plug

Commit message: Updating PESD1CAN part to new library path
Parts:
- D5: device Testing:SOT23-3 -> SparkFun-DiscreteSemi:SOT23-3
Changed lines of the file:
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@@
 <layer number="47" name="Measures" color="7" fill="1" visible="no" active="yes"/>
 <layer number="48" name="Document" color="7" fill="1" visible="no" active="yes"/>
-<layer number="49" name="Reference" color="7" fill="1" visible="yes" active="yes"/>
+<layer number="49" name="Reference" color="7" fill="1" visible="no" active="yes"/>
 <layer number="50" name="dxf" color="7" fill="1" visible="no" active="yes"/>
 <layer number="51" name="tDocu" color="6" fill="1" visible="yes" active="yes"/>
@@
 <element name="SJ5" library="SparkFun-Passives" package="PAD-JUMPER-3-2OF3_NC_BY_TRACE_YES_SILK_FULL_BOX" value="JUMPER-PAD-3-2OF3_NC_BY_TRACE_SMALL" x="26.67" y="46.0375" rot="R180"/>
 <element name="SJ6" library="SparkFun-Passives" package="PAD-JUMPER-3-2OF3_NC_BY_TRACE_YES_SILK_FULL_BOX" value="JUMPER-PAD-3-2OF3_NC_BY_TRACE_SMALL" x="21.2725" y="46.0375" rot="R180"/>
-<element name="D5" library="Testing" package="SOT23-3" value="PESD1CAN" x="14.605" y="38.1" rot="R180">
+<element name="D5" library="SparkFun-DiscreteSemi" package="SOT23-3" value="PESD1CAN" x="14.605" y="38.1" rot="R180">
 <attribute name="PROD_ID" value="DIO-12501" x="14.605" y="38.1" size="1.778" layer="27" font="vector" ratio="15" rot="R180" display="off"/>
 </element>
